File: BeagleBone-MSP430Cape/BeagleBone-MSP430Cape.sch (EAGLE design)
At the start: 2 parts

Commit message: schematic updates 05/07
Parts:
- added IC1: (no value), ic-package:DIL20S
- added SW1: (no value), SparkFun-Electromechanical:SW_DIP-2
Other:
- note added: "20 pin socket"
- note added: "Sets cape address"
- moved on the sheet: U$3
Changed lines of the file:
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@@
 <part name="GND2" library="SparkFun-Aesthetics" deviceset="GND" device=""/>
 <part name="U$3" library="TI_MSP430_v16" deviceset="G2X[1/5]2---N20" device=""/>
+<part name="IC1" library="ic-package" deviceset="DIL20" device="S"/>
+<part name="SW1" library="SparkFun-Electromechanical" deviceset="SW_DIP-2" device=""/>
 </parts>
 <sheets>
 <sheet>
 <plain>
-<text x="152.4" y="66.04" size="1.778" layer="91">Use MSP430G2253 in PDIP-20 package</text>
+<text x="170.18" y="2.54" size="1.778" layer="91">Use MSP430G2253 in PDIP-20 package</text>
+<text x="180.34" y="88.9" size="1.778" layer="91">20 pin socket</text>
+<text x="147.32" y="58.42" size="1.778" layer="91">Sets cape address</text>
 </plain>
 <instances>
@@
 <instance part="SUPPLY3" gate="G$1" x="10.16" y="66.04"/>
 <instance part="GND2" gate="1" x="22.86" y="0"/>
-<instance part="U$3" gate="G$1" x="175.26" y="88.9"/>
+<instance part="U$3" gate="G$1" x="193.04" y="25.4"/>
+<instance part="IC1" gate="G$1" x="190.5" y="106.68"/>
+<instance part="SW1" gate="G$1" x="154.94" y="66.04"/>
 </instances>
 <busses>
