File: BeagleBone-MSP430Cape/BeagleBone-MSP430Cape.sch (EAGLE design)
At the start: 4 parts

Commit message: updates 05/10/13
Parts:
- removed U$3: G2X[1/5]2---N20, TI_MSP430_v16:G2X[1/5]2---N20
- added C1, C2: 0.1 uF, SparkFun-Capacitors:CAP0805
- added R1: 10k, SparkFun-Resistors:RESISTOR0805-RES
- added R2, R3, R4: 4.75k, SparkFun-Resistors:RESISTOR0805-RES
- added R5, R6: 5.6k, SparkFun-Resistors:RESISTOR0805-RES
- added U$2: CAT24C256W, vttay03_custom:CAT24C256W
Connections:
- removed net I2C2_SCL: U$1.I2C2_SCL
- removed net I2C2_SDA: U$1.I2C2_SDA
- new net I2C_SCL: IC1.14, R5.1, U$1.I2C2_SCL, U$2.SCL
- new net I2C_SDA: IC1.15, R6.1, U$1.I2C2_SDA, U$2.SDA
- new net N$4: R2.1, U$2.A2
- new net N$5: R3.1, SW1.2, U$2.A1
- new net N$6: R4.1, SW1.1, U$2.A0
- new net WP_CTRL: R1.1, U$2.WP
- net 3.3V: now also C1.1, C2.1, IC1.1, R1.2, R2.2, R3.2, R4.2, R5.2, R6.2, U$2.VCC
- net GND: now also C1.2, C2.2, IC1.20, SW1.3, SW1.4, U$1.GND@4, U$2.GND
Other:
- note added: "MSP430G2553 Socket"
- note added: "Need actual DIP Switch Part No."
- note added: "Need to figure out how to tie WP back to Bone."
- note added: "Note: MSP430 has internal pullups for I2C bus."
- note removed: "20 pin socket"
- note removed: "Sets cape address"
- note removed: "Use MSP430G2253 in PDIP-20 package"
- moved on the sheet: IC1, SW1, U$1

Commit message: changes 05/12/13
Parts:
- added C3, C4, C5, C6, C7, C8, C9: 0.1 uF, SparkFun-Capacitors:CAP0805
- added D1: GREEN, SparkFun-LED:LED-GREEN0603
- added J1, J2: PINHD-1X10, adafruit:PINHD-1X10
- added JP1: RSTN_SEL, adafruit:PINHD-1X3
- added JP2: P2.0 SEL, SparkFun-Connectors:M02PTH
- added JP3: EEPROM_WP, SparkFun-Connectors:M02PTH
- added JP4: P2.1 SEL, SparkFun-Connectors:M02PTH
- added LED1: RED, SparkFun-LED:LED0603
- added LED2: GREEN, SparkFun-LED:LED0603
- added LED3: RGBLED5050, adafruit:RGBLED5050
- added R10, R11: 200, SparkFun-Resistors:RESISTOR0805-RES
- added R12, R13, R8: 130, SparkFun-Resistors:RESISTOR0805-RES
- added R14, R15: 0, SparkFun-Resistors:RESISTOR0805-RES
- added R7: 47k, SparkFun-Resistors:RESISTOR0805-RES
- added R9: 300, SparkFun-Resistors:RESISTOR0805-RES
- added S1: L_RSTN, switch-omron:10-XX
- added S2: USER, switch-omron:10-XX
- added U1: (no value), SparkFun-DigitalIC:TXB0104PWRSOIC14
- added U2: MAX232SOIC16, SparkFun-DigitalIC:MAX232SOIC16
- added X1: (no value), SparkFun-Connectors:DB9MALE
Connections:
- new net LED_BLUE_3_3V: U$1.GPIO2_1, U1.A3
- new net LED_BLUE_5V: R11.1, U1.B3
- new net LED_GREEN_3_3V: U$1.GPIO1_14, U1.A2
- new net LED_GREEN_5V: R10.1, U1.B2
- new net LED_RED_3_3V: U$1.GPIO0_26, U1.A1
- new net LED_RED_5V: R9.1, U1.B1
- new net MSP430I2C_SCL: IC1.14, J2.7, R14.2
- new net MSP430I2C_SDA: IC1.15, J2.6, R15.2
- new net N$10: JP4.2, R12.2
- new net N$11: LED2.A, R12.1
- new net N$19: D1.C, R8.2
- new net N$2: C5.2, U2.C1-
- new net N$20: LED3.RED_A, R9.2
- new net N$21: LED3.GREEN_A, R10.2
- new net N$22: LED3.BLUE_A, R11.2
- new net N$23: C8.1, U2.V+
- new net N$24: C5.1, U2.C1+
- new net N$27: C6.1, U2.C2+
- new net N$28: C6.2, U2.C2-
- new net N$3: C7.1, U2.V-
- new net N$7: LED1.A, R13.1
- new net N$8: JP2.2, R13.2
- new net P1.0: IC1.2, J1.2
- new net P1.3: IC1.5, J1.5
- new net P1.4: IC1.6, J1.6
- new net P1.5: IC1.7, J1.7
- new net P2.0: IC1.8, J1.8, JP2.1
- new net P2.1: IC1.9, J1.9, JP4.1
- new net P2.2: IC1.10, J1.10, S2.S, S2.S1
- new net P2.3: IC1.11, J2.10
- new net P2.4: IC1.12, J2.9
- new net P2.5: IC1.13, J2.8
- new net RSTN: IC1.16, J2.5, JP1.2, R7.1
- new net RSTN_BBONE: JP1.3, U$1.GPIO1_12
- new net RSTN_SWITCH: JP1.1, S1.S, S1.S1
- new net RXD: IC1.3, J1.3, U2.R1OUT
- new net RXD#: U2.R1IN, X1.2
- new net TEST/SBWTCK: IC1.17, J2.4
- new net TXD: IC1.4, J1.4, U2.T1IN
- new net TXD#: U2.T1OUT, X1.3
- new net XIN: J2.2
- new net XINR: IC1.19
- new net XOUT: J2.3
- new net XOUTR: IC1.18
- net 3.3V: now also C3.1, C9.1, D1.A, J1.1, R7.2, U1.OE, U1.VCCA, U2.VCC
- net 5V: now also C4.1, U1.VCCB
- net GND: now also C3.2, C4.2, C7.2, C8.2, C9.2, J2.1, JP3.2, LED1.C, LED2.C, LED3.BLUE_C, LED3.GREEN_C, LED3.RED_C, R8.1, S1.P, S1.P1, S2.P, S2.P1, U1.A4, U1.GND, U2.GND, U2.R2IN, U2.T2IN, X1.5
- net I2C_SCL: now also R14.1; no longer IC1.14
- net I2C_SDA: now also R15.1; no longer IC1.15
- net WP_CTRL: now also JP3.1
Other:
- note added: "0 ohm jumper connects MSP430 to I2C Bus."
- note added: "Digikey Part No. CT2092MS-ND"
- note added: "Note: Resistor values are based on 10 mA. Vf = 2V (Red), 3V (Blue), 3V (Green)"
- note added: "Pin compatible with MAX3232E (3.3V Part)."
- note added: "Shunt jumper enables EEPROM write."
- note added: "Shunt jumper will select reset source of MSP430."
- note added: "Shunt jumpers select whether LED(s) are driven."
- note added: "Use Digikey Part No. A35105-ND (Male Version) Confirm PCB footprint is for female (pins will need to be reversed on schematic if that's the case)"
- note added: "User button"
- note removed: "Need actual DIP Switch Part No."
- note removed: "Need to figure out how to tie WP back to Bone."
- moved on the sheet: C1, C2, IC1, R1, R2, R3, R4, R5, R6, SW1, U$2

Commit message: schematic/board updates 05/13
Parts:
- added LOGO1: OSHW-LOGOL, SparkFun-Aesthetics:OSHW-LOGOL
- renumbered LED1 to D2, LED2 to D3, LED3 to LED, U$2 to U3
Other:
- note added: "Add 5V PWR GOOD LED"
- note added: "Add pullup resistor?"
- note added: "PWR GOOD LED"
Changed lines of the file:
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@@
 <parts>
 <part name="U$1" library="adafruit" deviceset="BEAGLEBONE_OUTLINE" device=""/>
-<part name="U$2" library="vttay03_custom" deviceset="CAT24C256W" device=""/>
+<part name="U3" library="vttay03_custom" deviceset="CAT24C256W" device=""/>
 <part name="SUPPLY1" library="SparkFun-Aesthetics" deviceset="3.3V" device=""/>
 <part name="SUPPLY2" library="SparkFun-Aesthetics" deviceset="5V" device=""/>
@@
 <part name="S2" library="switch-omron" deviceset="10-XX" device="" value="USER"/>
 <part name="GND20" library="SparkFun-Aesthetics" deviceset="GND" device=""/>
-<part name="LED1" library="SparkFun-LED" deviceset="LED" device="0603" value="RED"/>
-<part name="LED2" library="SparkFun-LED" deviceset="LED" device="0603" value="GREEN"/>
+<part name="D2" library="SparkFun-LED" deviceset="LED" device="0603" value="RED"/>
+<part name="D3" library="SparkFun-LED" deviceset="LED" device="0603" value="GREEN"/>
 <part name="JP2" library="SparkFun-Connectors" deviceset="M02" device="PTH" value="P2.0 SEL"/>
 <part name="JP4" library="SparkFun-Connectors" deviceset="M02" device="PTH" value="P2.1 SEL"/>
@@
 <part name="R12" library="SparkFun-Resistors" deviceset="RESISTOR" device="0805-RES" value="130"/>
 <part name="R13" library="SparkFun-Resistors" deviceset="RESISTOR" device="0805-RES" value="130"/>
-<part name="LED3" library="adafruit" deviceset="RGBLED" device="5050"/>
+<part name="LED" library="adafruit" deviceset="RGBLED" device="5050"/>
 <part name="R14" library="SparkFun-Resistors" deviceset="RESISTOR" device="0805-RES" value="0"/>
 <part name="R15" library="SparkFun-Resistors" deviceset="RESISTOR" device="0805-RES" value="0"/>
+<part name="LOGO1" library="SparkFun-Aesthetics" deviceset="OSHW-LOGO" device="L"/>
 </parts>
 <sheets>
@@
 <text x="266.7" y="17.78" size="1.778" layer="91">Shunt jumpers select whether LED(s) are driven.</text>
 <text x="309.88" y="-2.54" size="1.778" layer="91">0 ohm jumper connects MSP430 to I2C Bus.</text>
+<text x="147.32" y="7.62" size="1.778" layer="91">Add pullup resistor?</text>
+<text x="162.56" y="101.6" size="1.778" layer="91">PWR GOOD LED</text>
+<text x="162.56" y="99.06" size="1.778" layer="91">Add 5V PWR GOOD LED</text>
 </plain>
 <instances>
 <instance part="U$1" gate="G$1" x="78.74" y="76.2"/>
-<instance part="U$2" gate="G$1" x="238.76" y="137.16"/>
+<instance part="U3" gate="G$1" x="238.76" y="137.16"/>
 <instance part="SUPPLY1" gate="G$1" x="124.46" y="71.12"/>
 <instance part="SUPPLY2" gate="G$1" x="132.08" y="71.12"/>
@@
 <instance part="S2" gate="1" x="152.4" y="17.78" rot="R270"/>
 <instance part="GND20" gate="1" x="139.7" y="7.62"/>
-<instance part="LED1" gate="G$1" x="261.62" y="17.78"/>
-<instance part="LED2" gate="G$1" x="274.32" y="2.54"/>
+<instance part="D2" gate="G$1" x="261.62" y="17.78"/>
+<instance part="D3" gate="G$1" x="274.32" y="2.54"/>
 <instance part="JP2" gate="G$1" x="299.72" y="30.48" rot="R180"/>
 <instance part="JP4" gate="G$1" x="299.72" y="10.16" rot="R180"/>
@@
 <instance part="R12" gate="G$1" x="284.48" y="7.62"/>
 <instance part="R13" gate="G$1" x="284.48" y="27.94"/>
-<instance part="LED3" gate="G$1" x="497.84" y="20.32" rot="R270"/>
+<instance part="LED" gate="G$1" x="497.84" y="20.32" rot="R270"/>
 <instance part="R14" gate="G$1" x="332.74" y="10.16"/>
 <instance part="R15" gate="G$1" x="332.74" y="2.54"/>
+<instance part="LOGO1" gate="G$1" x="142.24" y="157.48"/>
 </instances>
 <busses>
@@
 </segment>
 <segment>
-<pinref part="U$2" gate="G$1" pin="VCC"/>
+<pinref part="U3" gate="G$1" pin="VCC"/>
 <wire x1="251.46" y1="144.78" x2="302.26" y2="144.78" width="0.1524" layer="91"/>
 <pinref part="C1" gate="G$1" pin="1"/>
@@
 </segment>
 <segment>
-<pinref part="U$2" gate="G$1" pin="GND"/>
+<pinref part="U3" gate="G$1" pin="GND"/>
 <pinref part="GND1" gate="1" pin="GND"/>
 <wire x1="228.6" y1="129.54" x2="226.06" y2="129.54" width="0.1524" layer="91"/>
@@
 <segment>
 <pinref part="GND21" gate="1" pin="GND"/>
-<pinref part="LED2" gate="G$1" pin="C"/>
+<pinref part="D3" gate="G$1" pin="C"/>
 <wire x1="274.32" y1="-7.62" x2="274.32" y2="-2.54" width="0.1524" layer="91"/>
 </segment>
 <segment>
 <pinref part="GND22" gate="1" pin="GND"/>
-<pinref part="LED1" gate="G$1" pin="C"/>
+<pinref part="D2" gate="G$1" pin="C"/>
 <wire x1="261.62" y1="-7.62" x2="261.62" y2="12.7" width="0.1524" layer="91"/>
 </segment>
 <segment>
-<pinref part="LED3" gate="G$1" pin="RED_C"/>
+<pinref part="LED" gate="G$1" pin="RED_C"/>
 <wire x1="492.76" y1="15.24" x2="492.76" y2="7.62" width="0.1524" layer="91"/>
 <wire x1="492.76" y1="7.62" x2="497.84" y2="7.62" width="0.1524" layer="91"/>
@@
 <wire x1="497.84" y1="7.62" x2="502.92" y2="7.62" width="0.1524" layer="91"/>
 <wire x1="502.92" y1="7.62" x2="502.92" y2="0" width="0.1524" layer="91"/>
-<pinref part="LED3" gate="G$1" pin="BLUE_C"/>
+<pinref part="LED" gate="G$1" pin="BLUE_C"/>
 <wire x1="502.92" y1="7.62" x2="502.92" y2="15.24" width="0.1524" layer="91"/>
 <junction x="502.92" y="7.62"/>
-<pinref part="LED3" gate="G$1" pin="GREEN_C"/>
+<pinref part="LED" gate="G$1" pin="GREEN_C"/>
 <wire x1="497.84" y1="15.24" x2="497.84" y2="7.62" width="0.1524" layer="91"/>
 <junction x="497.84" y="7.62"/>
@@
 </segment>
 <segment>
-<pinref part="U$2" gate="G$1" pin="SCL"/>
+<pinref part="U3" gate="G$1" pin="SCL"/>
 <wire x1="251.46" y1="134.62" x2="266.7" y2="134.62" width="0.1524" layer="91"/>
 <label x="254" y="134.62" size="1.778" layer="95"/>
@@
 </segment>
 <segment>
-<pinref part="U$2" gate="G$1" pin="SDA"/>
+<pinref part="U3" gate="G$1" pin="SDA"/>
 <wire x1="251.46" y1="129.54" x2="274.32" y2="129.54" width="0.1524" layer="91"/>
 <label x="254" y="129.54" size="1.778" layer="95"/>
@@
 <segment>
 <pinref part="R1" gate="G$1" pin="1"/>
-<pinref part="U$2" gate="G$1" pin="WP"/>
+<pinref part="U3" gate="G$1" pin="WP"/>
 <wire x1="287.02" y1="139.7" x2="281.94" y2="139.7" width="0.1524" layer="91"/>
 <wire x1="281.94" y1="139.7" x2="251.46" y2="139.7" width="0.1524" layer="91"/>
@@
 <pinref part="R2" gate="G$1" pin="1"/>
 <wire x1="208.28" y1="152.4" x2="208.28" y2="134.62" width="0.1524" layer="91"/>
-<pinref part="U$2" gate="G$1" pin="A2"/>
+<pinref part="U3" gate="G$1" pin="A2"/>
 <wire x1="208.28" y1="134.62" x2="228.6" y2="134.62" width="0.1524" layer="91"/>
 </segment>
@@
 <pinref part="R3" gate="G$1" pin="1"/>
 <wire x1="215.9" y1="152.4" x2="215.9" y2="139.7" width="0.1524" layer="91"/>
-<pinref part="U$2" gate="G$1" pin="A1"/>
+<pinref part="U3" gate="G$1" pin="A1"/>
 <wire x1="215.9" y1="139.7" x2="228.6" y2="139.7" width="0.1524" layer="91"/>
 <pinref part="SW1" gate="G$1" pin="2"/>
@@
 <pinref part="R4" gate="G$1" pin="1"/>
 <wire x1="223.52" y1="152.4" x2="223.52" y2="144.78" width="0.1524" layer="91"/>
-<pinref part="U$2" gate="G$1" pin="A0"/>
+<pinref part="U3" gate="G$1" pin="A0"/>
 <wire x1="223.52" y1="144.78" x2="228.6" y2="144.78" width="0.1524" layer="91"/>
 <pinref part="SW1" gate="G$1" pin="1"/>
@@
 <pinref part="R9" gate="G$1" pin="2"/>
 <wire x1="452.12" y1="35.56" x2="492.76" y2="35.56" width="0.1524" layer="91"/>
-<pinref part="LED3" gate="G$1" pin="RED_A"/>
+<pinref part="LED" gate="G$1" pin="RED_A"/>
 <wire x1="492.76" y1="35.56" x2="492.76" y2="25.4" width="0.1524" layer="91"/>
 </segment>
@@
 <pinref part="R10" gate="G$1" pin="2"/>
 <wire x1="497.84" y1="33.02" x2="464.82" y2="33.02" width="0.1524" layer="91"/>
-<pinref part="LED3" gate="G$1" pin="GREEN_A"/>
+<pinref part="LED" gate="G$1" pin="GREEN_A"/>
 <wire x1="497.84" y1="33.02" x2="497.84" y2="25.4" width="0.1524" layer="91"/>
 </segment>
@@
 <segment>
 <pinref part="R11" gate="G$1" pin="2"/>
-<pinref part="LED3" gate="G$1" pin="BLUE_A"/>
+<pinref part="LED" gate="G$1" pin="BLUE_A"/>
 <wire x1="477.52" y1="30.48" x2="502.92" y2="30.48" width="0.1524" layer="91"/>
 <wire x1="502.92" y1="30.48" x2="502.92" y2="25.4" width="0.1524" layer="91"/>
@@
 <net name="N$7" class="0">
 <segment>
-<pinref part="LED1" gate="G$1" pin="A"/>
+<pinref part="D2" gate="G$1" pin="A"/>
 <wire x1="261.62" y1="20.32" x2="261.62" y2="27.94" width="0.1524" layer="91"/>
 <pinref part="R13" gate="G$1" pin="1"/>
@@
 <segment>
 <pinref part="R12" gate="G$1" pin="1"/>
-<pinref part="LED2" gate="G$1" pin="A"/>
+<pinref part="D3" gate="G$1" pin="A"/>
 <wire x1="279.4" y1="7.62" x2="274.32" y2="7.62" width="0.1524" layer="91"/>
 <wire x1="274.32" y1="7.62" x2="274.32" y2="5.08" width="0.1524" layer="91"/>
