File: BeagleBone-MSP430Cape/BeagleBone-MSP430Cape.brd (EAGLE design)
At the start: 71.8 x 54.6 mm, 43 parts, among them J1 PINHD-1X10, J2 PINHD-1X10, U2 MAX232SOIC16

Commit message: schematic/board updates 05/13
Parts:
- removed LED1: RED, SparkFun-LED:LED-0603
- removed LED2: GREEN, SparkFun-LED:LED-0603
- removed LED3: RGBLED5050, adafruit:RGBLED5050
- removed U$2: CAT24C256W, vttay03_custom:SO08
- added D2: RED, SparkFun-LED:LED-0603
- added D3: GREEN, SparkFun-LED:LED-0603
- added LED: RGBLED5050, adafruit:RGBLED5050
- added LOGO1: OSHW-LOGOL, SparkFun-Aesthetics:OSHW-LOGO-L
- added U3: CAT24C256W, vttay03_custom:SO08
- moved C5 13.6 mm to (26.7, 7.62), turned to 0 degrees
- moved C9 12.7 mm to (24.8, 18.4), turned to 0 degrees
- moved C7 12.6 mm to (15.9, 8.26), turned to 270 degrees
- moved R11 10.9 mm to (59.1, 17.1), flipped to the top, turned to 270 degrees
- moved R10 9.67 mm to (64.1, 17.1), flipped to the top, turned to 270 degrees
- moved C8 9.38 mm to (23.5, 8.26), turned to 270 degrees
- moved R9 8.98 mm to (61.6, 17.1), flipped to the top, turned to 270 degrees
- moved C1 8.91 mm to (55.2, 41.3), flipped to the top
- moved C6 8.64 mm to (19.7, 7.62), turned to 0 degrees
- moved R1 4.84 mm to (55.9, 47.0), flipped to the top, turned to 180 degrees
- moved U2 3.18 mm to (21.6, 14.0), turned to 0 degrees
- moved R5 2.29 mm to (61.0, 47.0), flipped to the top
- moved R6 2.01 mm to (64.8, 47.0), flipped to the top
- moved SW1 1.91 mm to (59.7, 24.8)
- moved JP4 1.42 mm to (41.9, 15.2)
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Connections:
- net 3.3V: now also U3.8; no longer U$2.8
- net GND: now also D2.C, D3.C, LED.4, LED.5, LED.6, U3.4; no longer LED1.C, LED2.C, LED3.4, LED3.5, LED3.6, U$2.4
- net I2C_SCL: now also U3.6; no longer U$2.6
- net I2C_SDA: now also U3.5; no longer U$2.5
- net N$11: now also D3.A; no longer LED2.A
- net N$20: now also LED.2; no longer LED3.2
- net N$21: now also LED.1; no longer LED3.1
- net N$22: now also LED.3; no longer LED3.3
- net N$4: now also U3.3; no longer U$2.3
- net N$5: now also U3.2; no longer U$2.2
- net N$6: now also U3.1; no longer U$2.1
- net N$7: now also D2.A; no longer LED1.A
- net WP_CTRL: now also U3.7; no longer U$2.7
Routing:
- net GND: track 363.0 -> 314.7 mm
- net LED_BLUE_5V: track 49.9 -> 19.8 mm, vias 0 -> 1
- net N$5: track 41.2 -> 23.1 mm
- net RXD#: track 39.3 -> 21.3 mm
- net 5V: track 49.1 -> 61.3 mm, vias 1 -> 0
- net N$11: track 10.3 -> 2.80 mm, vias 1 -> 0
- net I2C_SDA: track 50.0 -> 57.5 mm, vias 1 -> 0
- net N$7: track 9.90 -> 2.81 mm, vias 1 -> 0
- net I2C_SCL: track 47.4 -> 41.0 mm
- net TXD#: track 30.6 -> 36.1 mm
- net RXD: track 19.8 -> 14.6 mm
- net N$4: track 8.25 -> 3.75 mm, vias 1 -> 0
- net N$3: track 3.18 -> 7.62 mm, vias 0 -> 2
- net LED_RED_5V: track 17.1 -> 12.7 mm, vias 2 -> 1
- net 3.3V: track 227.0 -> 229.7 mm, vias 3 -> 1
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Other:
- board text added: "MSP430 Cape (c) vttay03 05/2013 Rev -"
